Commit message: first commit

File: rockbreaker_description/urdf/rockbreaker_arm.urdf.xacro (robot description, xacro)
@@ -1,13 +1,14 @@
 <?xml version="1.0"?>
 <robot xmlns:xacro="http://www.ros.org/wiki/xacro" name="rockbreaker_arm">
-  <xacro:arg name="gpu" default="false"/>
+  <xacro:arg name="gpu" default="true"/>
   <xacro:property name="gpu" value="$(arg gpu)" />
-  <xacro:arg name="organize_cloud" default="false"/>
+  <xacro:arg name="organize_cloud" default="true"/>
   <xacro:property name="organize_cloud" value="$(arg organize_cloud)" />
   <xacro:property name="M_PI" value="3.1415926535897931" />
-  <xacro:property name="damping_value" value="10" />
+  <xacro:property name="damping_value" value="1.0" />
   <xacro:property name="friction_value" value="0.1" />
    <!-- Import all Gazebo-customization elements, including Gazebo colors -->
-  <xacro:include filename="$(find rockbreaker_arm_simulator)/rockbreaker_description/urdf/rockbreaker_arm.gazebo" />
+  <xacro:include filename="$(find rockbreaker_arm_simulator)/rockbreaker_description/urdf/rockbreaker_arm.gazebo"/>
+  <xacro:include filename="$(find rockbreaker_arm_simulator)/rockbreaker_arm_gazebo/models/kinect/model.sdf"/>
   <xacro:macro name="box_inertia" params="x y z mass">
     <!-- <inertial>
@@ -24,23 +25,23 @@
     <parent link="world" />
     <child link="rockbreaker_base" />
-     <origin xyz="0 0 -0.2" />
+     <origin xyz="-3 -3 15.756649" rpy="0 0 1.571"/>
   </joint>
   <!-- Base Fija -->
   <link name="rockbreaker_base" >
     <visual>
-      <origin xyz="0 0 0.2" rpy="0 0 0"/>
-      <geometry>
-        <!--<mesh filename = "file:///home/kyungki/workspace/catkin_ws/src/velodyne_simulator/velodyne_description/meshes/excavator-1.dae"/>-->
-        <mesh filename="package://rockbreaker_arm_simulator/rockbreaker_description/meshes/base_fija.dae" scale="1 1 1"/>
-      </geometry>
-    </visual>
-    <collision>
-      <origin xyz="0 0 0.2" rpy="0 0 0"/>
-      <geometry>
-        <mesh filename="package://rockbreaker_arm_simulator/rockbreaker_description/meshes/base_fija.dae" scale="1 1 1"/>
-      </geometry>
-    </collision>
-    <inertial>
-      <origin xyz="1.25 1.25 0.5"/>
+      <origin xyz="0 0 0" rpy="0 0 0"/>
+      <geometry>
+        <!--<mesh filename = "file:///home/kyungki/workspace/catkin_ws/src/velodyne_simulator/velodyne_description/meshes/excavator-1.dae"/>-->
+        <mesh filename="package://rockbreaker_arm_simulator/rockbreaker_description/meshes/basefija.dae" scale="1 1 1"/>
+      </geometry>
+    </visual>
+    <collision>
+      <origin xyz="0 0 0" rpy="0 0 0"/>
+      <geometry>
+        <mesh filename="package://rockbreaker_arm_simulator/rockbreaker_description/meshes/basefija.dae" scale="1 1 1"/>
+      </geometry>
+    </collision>
+    <inertial>
+      <origin xyz="0 0 0.3"/>
       <mass value="1000"/>
       <xacro:box_inertia x="2.5" y="2.5" z="0.5" mass="1000"/>
@@ -50,5 +51,5 @@
   <link name="rockbreaker_baserotatoria" >
     <visual>
-      <origin xyz="0 0 0" rpy="0 0 59.7"/>
+      <origin xyz="0 0 -0.2" rpy="0 0 59.7"/>
       <geometry>
         <!-- <mesh filename = "file:///home/kyungki/workspace/catkin_ws/src/velodyne_simulator/velodyne_description/meshes/excavator-1.dae"/> -->
@@ -57,5 +58,5 @@
     </visual>
     <collision>
-      <origin xyz="0 0 0" rpy="0 0 59.7"/>
+      <origin xyz="0 0 -0.2" rpy="0 0 59.7"/>
       <geometry>
         <mesh filename="package://rockbreaker_arm_simulator/rockbreaker_description/meshes/base_rotatoria.dae" scale="0.1 0.1 0.1"/>
@@ -63,5 +64,5 @@
     </collision>
     <inertial>
-      <origin xyz="0 0 0.4" rpy="0 0 59.7"/>
+      <origin xyz="0 0 0.2" rpy="0 0 59.7"/>
       <mass value="400"/>
      <xacro:box_inertia x="1.4" y="1.4" z="1.1" mass="400"/>
@@ -71,5 +72,5 @@
   <link name="brazo_a" >
     <visual>
-      <origin xyz="0 0 0" rpy="0 0.6 1.57"/>
+      <origin xyz="0 0 -0.2" rpy="0 0.6 1.57"/>
       <geometry> -->
         <!--<mesh filename = "file:///home/kyungki/workspace/catkin_ws/src/velodyne_simulator/velodyne_description/meshes/excavator-1.dae"/>-->
@@ -78,5 +79,5 @@
     </visual>
     <collision>
-      <origin xyz="0 0 0" rpy="0 0.6 1.57"/>
+      <origin xyz="0 0 -0.2" rpy="0 0.6 1.57"/>
       <geometry>
            <mesh filename="package://rockbreaker_arm_simulator/rockbreaker_description/meshes/BrazoA_rockbreaker.dae" scale="1 1 1"/>
@@ -84,7 +85,7 @@
     </collision>
     <inertial>
-      <origin xyz="-0.4 -3.0 3.4" rpy="0 0.6 1.57"/>
-      <mass value="100"/>
-       <xacro:box_inertia x="7.4" y="1" z="1.5" mass="100"/>
+      <origin xyz="-0.4 -3.0 3.2" rpy="0 0.6 1.57"/>
+      <mass value="160"/>
+       <xacro:box_inertia x="7.8" y="1.5" z="1.5" mass="100"/>
      </inertial>
   </link>
@@ -92,5 +93,5 @@
   <link name="brazo_b" >
     <visual>
-      <origin xyz="0 0 0" rpy="0 0.6 1.57"/>
+      <origin xyz="0 0 -0.2" rpy="0 0.6 1.57"/>
       <geometry>
         <!--<mesh filename = "file:///home/kyungki/workspace/catkin_ws/src/velodyne_simulator/velodyne_description/meshes/excavator-1.dae"/>-->
@@ -99,5 +100,5 @@
     </visual>
     <collision>
-      <origin xyz="0 0 0" rpy="0 0.6 1.57"/>
+      <origin xyz="0 0 -0.2" rpy="0 0.6 1.57"/>
       <geometry>
         <mesh filename="package://rockbreaker_arm_simulator/rockbreaker_description/meshes/BrazoB_rockbreaker.dae" scale="1 1 1"/>
@@ -105,5 +106,5 @@
     </collision>
     <inertial>
-      <origin xyz="0.5 -4.0 3.0" rpy="0 0.6 1.57"/>
+      <origin xyz="0.5 -4.0 2.8" rpy="0 0.6 1.57"/>
       <mass value="80"/>
      <xacro:box_inertia x="6.0" y="1" z="1.5" mass="80"/>
@@ -113,5 +114,5 @@
   <link name="h_hammer" >
     <visual>
-      <origin xyz="0 0 0" rpy="0 1.57 1.57"/>
+      <origin xyz="0 0 -0.2" rpy="0 1.57 1.57"/>
       <geometry>
         <!--<mesh filename = "file:///home/kyungki/workspace/catkin_ws/src/velodyne_simulator/velodyne_description/meshes/excavator-1.dae"/>-->
@@ -120,5 +121,5 @@
     </visual>
     <collision>
-      <origin xyz="0 0 0" rpy="0 1.57 1.57"/>
+      <origin xyz="0 0 -0.2" rpy="0 1.57 1.57"/>
       <geometry>
          <mesh filename="package://rockbreaker_arm_simulator/rockbreaker_description/meshes/Hydraulic_Hammer.dae" scale="1 1 1"/>
@@ -127,8 +128,70 @@
     <inertial>
       <origin xyz="-0.4 -1.5 0.2" rpy="0 1.57 1.57"/>
-      <mass value="50"/>
+      <mass value="40"/>
      <xacro:box_inertia x="1.0" y="1.3" z="2.3" mass="50"/>
      </inertial>
   </link>
+  <!-- <link name="base_ir_front">
+    <collision>
+      <origin xyz="0 0 0" rpy="0 0 0"/>
+      <geometry>
+        <box size="0.01 0.01 0.01"/>
+      </geometry>
+    </collision>
+    <visual>
+      <origin xyz="0 0 0" rpy="0 0 0"/>
+      <geometry>
+        <box size="0.01 0.01 0.01"/>
+      </geometry>
+    </visual>
+    <inertial>
+      <mass value="1e-5" />
+      <origin xyz="0 0 0" rpy="0 0 0"/>
+      <inertia ixx="1e-6" ixy="0" ixz="0" iyy="1e-6" iyz="0"      izz="1e-6" />
+    </inertial>
+  </link>
+  <gazebo reference="base_ir_front">
+   <sensor type="ray" name="Sonar">
+      <pose>0 0 0 0 0 0</pose>
+      <visualize>true</visualize>
+      <update_rate>20</update_rate>
+      <ray>
+         <scan>
+            <horizontal>
+               <samples>10</samples>
+               <resolution>1</resolution>
+               <min_angle>-0.25835</min_angle>
+               <max_angle>0.25835</max_angle>
+            </horizontal>
+            <vertical>
+               <samples>10</samples>
+               <resolution>1</resolution>
+               <min_angle>-0.25835</min_angle>
+               <max_angle>0.25835</max_angle>
+            </vertical>
+         </scan>
+         <range>
+            <min>0.01</min>
+            <max>7</max>
+            <resolution>0.01</resolution>
+         </range>
+      </ray>
+      <plugin filename="libgazebo_ros_range.so" name="gazebo_ros_range">
+         <gaussianNoise>0.005</gaussianNoise>
+         <alwaysOn>true</alwaysOn>
+         <updateRate>20</updateRate>
+         <topicName>/sensor</topicName>
+         <frameName>base_ir_front</frameName>
+         <radiation>ultrasound</radiation>
+         <fov>0.4967</fov>
+      </plugin>
+    </sensor>
+  </gazebo>
+  <joint name="ir_front_joint" type="fixed">
+    <axis xyz="0 0 0" />
+    <origin rpy="1.57 0 0" xyz="0 0 0" />
+    <parent link="brazo_a"/>
+    <child link="base_ir_front"/>
+  </joint> -->
    <!-- Hydraulic Hammer Punta -->
   <!-- <link name="h_punta" >
@@ -156,13 +219,13 @@
   <joint name="joint_base_rockbreaker" type="revolute" >
     <axis xyz="0 0 1"/>
-    <limit effort="1000000" lower="-1.57" upper="1.57" velocity="100"/>
+    <limit effort="1000000" lower="-1.57" upper="1.57" velocity="10"/>
     <parent link="rockbreaker_base" />
     <child link="rockbreaker_baserotatoria"  />
-    <origin xyz="1.1 1.071 1.1 " rpy="0 0 0" />
+    <origin xyz="0 0 1.1 " rpy="0 0 0" />
     <dynamics damping="${damping_value}" friction="${friction_value}"/>
   </joint>
   <joint name="joint_brazoa" type="revolute" >
     <axis xyz="1 0 0"/>
-    <limit effort="10" lower="-3.1415" upper="3.1415" velocity="1"/>
+    <limit effort="1000000" lower="-3.14" upper="3.14" velocity="10"/>
     <parent link="rockbreaker_baserotatoria" />
     <child link="brazo_a" />
@@ -172,5 +235,5 @@
   <joint name="joint_brazob" type="revolute" >
     <axis xyz="1 0 0"/>
-    <limit effort="10" lower="-3.1415" upper="3.1415" velocity="1"/>
+    <limit effort="100000" lower="-3.14" upper="3.14" velocity="10"/>
     <parent link="brazo_a" />
     <child link="brazo_b" />
@@ -180,5 +243,5 @@
   <joint name="joint_hammer" type="revolute" >
     <axis xyz="1 0 0"/>
-    <limit effort="10" lower="0" upper="3.1415" velocity="1"/>
+    <limit effort="100000" lower="-3.14" upper="3.14" velocity="10"/>
     <parent link="brazo_b" />
     <child link="h_hammer" />
@@ -203,5 +266,5 @@
     </actuator>
   </transmission>
-  <!-- <transmission name="tran2">
+  <transmission name="tran2">
     <type>transmission_interface/SimpleTransmission</type>
     <joint name="joint_brazoa">
@@ -223,5 +286,5 @@
     </actuator>
   </transmission>
-   <transmission name="tran4">
+  <transmission name="tran4">
     <type>transmission_interface/SimpleTransmission</type>
     <joint name="joint_hammer">
@@ -232,5 +295,5 @@
       <mechanicalReduction>1</mechanicalReduction>
     </actuator>
-  </transmission> -->
+  </transmission>
   <!--
   <xacro:include filename="$(find velodyne_description)/urdf/VLP-16.urdf.xacro"/>
@@ -240,5 +303,8 @@
   -->
   <!-- <xacro:include filename=rockbreaker)/urdf/HDL-32E.urdf.xacro"/> -->
-  <!--<xacro:include filename="$(find velodyne_description)/urdf/camera.urdf.xacro"/>-->
+  <!-- <xacro:include filename="$(find lidar_description)/urdf/OS0-64.urdf.xacro"/>
+   <xacro:OS0-64 parent="rockbreaker_base" name="os0_sensor" topic="/os0_cloud_node/points"  hz="10" samples="512" >
+    <origin xyz="3 -13 0" rpy="0 0 1.57" />
+  </xacro:OS0-64> -->
   <!-- <xacro:include filename=rockbreaker)/urdf/stereo_camera.urdf.xacro"/>
   <xacro:include filename=rockbreaker)/urdf/VLP-16.urdf.xacro"/>
@@ -260,4 +326,74 @@
   </xacro:camera_sensor>
   -->
-   <!-- ros_control plugin -->
+  <!-- <link name="camera_link">
+    <visual>
+      <origin xyz="0 0 0" rpy="0 0 0"/>
+      <geometry>
+        <box size="1 1 1"/>
+      </geometry>
+    </visual>
+    <collision>
+      <origin xyz="0 0 0" rpy="0 0 0"/>
+      <geometry>
+        <box size="1 1 1"/>
+      </geometry>
+    </collision>
+    <inertial>
+      <origin xyz="0 0 0" rpy="0 0 0"/>
+      <mass value="0.035"/>
+      <inertia ixx="0.001"  ixy="0"  ixz="0" iyy="0.001" iyz="0" izz="0.001" />
+    </inertial>
+  </link>
+  <joint name="camera_joint" type="fixed">
+    <parent link="rockbreaker_baserotatoria"/>
+    <child link="camera_link"/>
+    <origin xyz="1 1 1" rpy="0 0 0"/>
+  </joint>
+  <link name="camera_depth_frame"/>
+  <joint name="camera_depth_joint" type="fixed">
+    <origin xyz="0 0 0" rpy="${-pi/2} 0 ${-pi/2}"/>
+    <parent link="camera_link"/>
+    <child link="camera_depth_frame"/>
+  </joint>
+  <gazebo reference="camera_link">
+  <sensor name="depth_camera" type="depth">
+    <update_rate>20</update_rate>
+    <camera>
+      <horizontal_fov>1.047198</horizontal_fov>
+      <image>
+        <width>640</width>
+        <height>480</height>
+        <format>R8G8B8</format>
+      </image>
+      <clip>
+        <near>0.05</near>
+        <far>3</far>
+      </clip>
+    </camera>
+    <plugin name="depth_camera_controller" filename="libgazebo_ros_openni_kinect.so">
+      <baseline>0.2</baseline>
+      <alwaysOn>true</alwaysOn>
+      <updateRate>1.0</updateRate>
+      <cameraName>kine_ir</cameraName>
+      <imageTopicName>/kine/color/image_raw</imageTopicName>
+      <cameraInfoTopicName>/kine/color/camera_info</cameraInfoTopicName>
+      <depthImageTopicName>/kine/depth/image_raw</depthImageTopicName>
+      <depthImageInfoTopicName>/kine/depth/camera_info</depthImageInfoTopicName>
+      <pointCloudTopicName>/kine/depth/points</pointCloudTopicName>
+      <frameName>kine_frame</frameName>
+      <pointCloudCutoff>0.5</pointCloudCutoff>
+      <pointCloudCutoffMax>3.0</pointCloudCutoffMax>
+      <distortionK1>0.00000001</distortionK1>
+      <distortionK2>0.00000001</distortionK2>
+      <distortionK3>0.00000001</distortionK3>
+      <distortionT1>0.00000001</distortionT1>
+      <distortionT2>0.00000001</distortionT2>
+      <CxPrime>0</CxPrime>
+      <Cx>0</Cx>
+      <Cy>0</Cy>
+      <focalLength>0</focalLength>
+      <hackBaseline>0</hackBaseline>
+    </plugin>
+  </sensor>
+</gazebo> -->
 </robot>

Commit message: Update rockbreaker_arm.urdf.xacro

File: rockbreaker_description/urdf/rockbreaker_arm.urdf.xacro (robot description, xacro)
@@ -32,5 +32,4 @@
       <origin xyz="0 0 0" rpy="0 0 0"/>
       <geometry>
-        <!--<mesh filename = "file:///home/kyungki/workspace/catkin_ws/src/velodyne_simulator/velodyne_description/meshes/excavator-1.dae"/>-->
         <mesh filename="package://rockbreaker_arm_simulator/rockbreaker_description/meshes/basefija.dae" scale="1 1 1"/>
       </geometry>
