Commit message: inserta Mensaje aquí.

File: rockbreaker_description/urdf/rockbreaker_arm.urdf.xacro (robot description, xacro)
@@ -8,5 +8,5 @@
   <xacro:property name="damping_value" value="1.0" />
   <xacro:property name="friction_value" value="0.1" />
-   <!-- Import all Gazebo-customization elements, including Gazebo colors -->
+  <!-- Import all Gazebo-customization elements, including Gazebo colors -->
   <xacro:include filename="$(find rockbreaker_arm_simulator)/rockbreaker_description/urdf/rockbreaker_arm.gazebo"/>
   <xacro:include filename="$(find rockbreaker_arm_simulator)/rockbreaker_arm_gazebo/models/kinect/model.sdf"/>
@@ -19,5 +19,5 @@
     <!-- </inertial> -->
   </xacro:macro>
- <!-- Base Fija -->
+  <!-- Base Fija -->
   <link name="world" />
   <!-- Base Link -->
@@ -32,5 +32,4 @@
       <origin xyz="0 0 0" rpy="0 0 0"/>
       <geometry>
-        <!--<mesh filename = "file:///home/kyungki/workspace/catkin_ws/src/velodyne_simulator/velodyne_description/meshes/excavator-1.dae"/>-->
         <mesh filename="package://rockbreaker_arm_simulator/rockbreaker_description/meshes/basefija.dae" scale="1 1 1"/>
       </geometry>
@@ -51,12 +50,11 @@
   <link name="rockbreaker_baserotatoria" >
     <visual>
-      <origin xyz="0 0 -0.2" rpy="0 0 59.7"/>
-      <geometry>
-        <!-- <mesh filename = "file:///home/kyungki/workspace/catkin_ws/src/velodyne_simulator/velodyne_description/meshes/excavator-1.dae"/> -->
+      <origin xyz="0 0 -0.2" rpy="0 0 3.14"/>
+      <geometry>
         <mesh filename="package://rockbreaker_arm_simulator/rockbreaker_description/meshes/base_rotatoria.dae" scale="0.1 0.1 0.1"/>
       </geometry>
     </visual>
     <collision>
-      <origin xyz="0 0 -0.2" rpy="0 0 59.7"/>
+      <origin xyz="0 0 -0.2" rpy="0 0 3.14"/>
       <geometry>
         <mesh filename="package://rockbreaker_arm_simulator/rockbreaker_description/meshes/base_rotatoria.dae" scale="0.1 0.1 0.1"/>
@@ -64,5 +62,5 @@
     </collision>
     <inertial>
-      <origin xyz="0 0 0.2" rpy="0 0 59.7"/>
+      <origin xyz="0 0 0.2" rpy="0 0 1.57"/>
       <mass value="400"/>
      <xacro:box_inertia x="1.4" y="1.4" z="1.1" mass="400"/>
@@ -73,6 +71,5 @@
     <visual>
       <origin xyz="0 0 -0.2" rpy="0 0.6 1.57"/>
-      <geometry> -->
-        <!--<mesh filename = "file:///home/kyungki/workspace/catkin_ws/src/velodyne_simulator/velodyne_description/meshes/excavator-1.dae"/>-->
+      <geometry>
         <mesh filename="package://rockbreaker_arm_simulator/rockbreaker_description/meshes/BrazoA_rockbreaker.dae" scale="1 1 1"/>
       </geometry>
@@ -95,5 +92,4 @@
       <origin xyz="0 0 -0.2" rpy="0 0.6 1.57"/>
       <geometry>
-        <!--<mesh filename = "file:///home/kyungki/workspace/catkin_ws/src/velodyne_simulator/velodyne_description/meshes/excavator-1.dae"/>-->
         <mesh filename="package://rockbreaker_arm_simulator/rockbreaker_description/meshes/BrazoB_rockbreaker.dae" scale="1 1 1"/>
       </geometry>
@@ -116,5 +112,4 @@
       <origin xyz="0 0 -0.2" rpy="0 1.57 1.57"/>
       <geometry>
-        <!--<mesh filename = "file:///home/kyungki/workspace/catkin_ws/src/velodyne_simulator/velodyne_description/meshes/excavator-1.dae"/>-->
         <mesh filename="package://rockbreaker_arm_simulator/rockbreaker_description/meshes/Hydraulic_Hammer.dae" scale="1 1 1"/>
       </geometry>
@@ -129,95 +124,11 @@
       <origin xyz="-0.4 -1.5 0.2" rpy="0 1.57 1.57"/>
       <mass value="40"/>
-     <xacro:box_inertia x="1.0" y="1.3" z="2.3" mass="50"/>
-     </inertial>
-  </link>
-  <!-- <link name="base_ir_front">
-    <collision>
-      <origin xyz="0 0 0" rpy="0 0 0"/>
-      <geometry>
-        <box size="0.01 0.01 0.01"/>
-      </geometry>
-    </collision>
-    <visual>
-      <origin xyz="0 0 0" rpy="0 0 0"/>
-      <geometry>
-        <box size="0.01 0.01 0.01"/>
-      </geometry>
-    </visual>
-    <inertial>
-      <mass value="1e-5" />
-      <origin xyz="0 0 0" rpy="0 0 0"/>
-      <inertia ixx="1e-6" ixy="0" ixz="0" iyy="1e-6" iyz="0"      izz="1e-6" />
-    </inertial>
-  </link>
-  <gazebo reference="base_ir_front">
-   <sensor type="ray" name="Sonar">
-      <pose>0 0 0 0 0 0</pose>
-      <visualize>true</visualize>
-      <update_rate>20</update_rate>
-      <ray>
-         <scan>
-            <horizontal>
-               <samples>10</samples>
-               <resolution>1</resolution>
-               <min_angle>-0.25835</min_angle>
-               <max_angle>0.25835</max_angle>
-            </horizontal>
-            <vertical>
-               <samples>10</samples>
-               <resolution>1</resolution>
-               <min_angle>-0.25835</min_angle>
-               <max_angle>0.25835</max_angle>
-            </vertical>
-         </scan>
-         <range>
-            <min>0.01</min>
-            <max>7</max>
-            <resolution>0.01</resolution>
-         </range>
-      </ray>
-      <plugin filename="libgazebo_ros_range.so" name="gazebo_ros_range">
-         <gaussianNoise>0.005</gaussianNoise>
-         <alwaysOn>true</alwaysOn>
-         <updateRate>20</updateRate>
-         <topicName>/sensor</topicName>
-         <frameName>base_ir_front</frameName>
-         <radiation>ultrasound</radiation>
-         <fov>0.4967</fov>
-      </plugin>
-    </sensor>
-  </gazebo>
-  <joint name="ir_front_joint" type="fixed">
-    <axis xyz="0 0 0" />
-    <origin rpy="1.57 0 0" xyz="0 0 0" />
-    <parent link="brazo_a"/>
-    <child link="base_ir_front"/>
-  </joint> -->
-   <!-- Hydraulic Hammer Punta -->
-  <!-- <link name="h_punta" >
-    <visual>
-      <origin xyz="0 0 0" rpy="-0.6 0 0"/>
-      <geometry> -->
-        <!--<mesh filename = "file:///home/kyungki/workspace/catkin_ws/src/velodyne_simulator/velodyne_description/meshes/excavator-1.dae"/>-->
-        <!-- <mesh filename="package://rockbreaker_arm_simulator/rockbreaker_description/meshes/Hydraulic_Hammer.dae" scale="1 1 1"/>
-      </geometry>
-    </visual>
-    <collision>
-      <origin xyz="0 0 0" rpy="-0.6 0 0"/>
-      <geometry>
-        <mesh filename="package://rockbreaker_arm_simulator/rockbreaker_description/meshes/Hydraulic_Hammer.dae" scale="1 1 1"/>
-      </geometry>
-    </collision>
-    <inertial>
-      <origin xyz="0 0 0"/>
-      <mass value="5"/>
-      <inertia ixx="3.0" ixy="0.0" ixz="0.0"
-               iyy="3.0" iyz="0.0"
-               izz="3.0" />
-    </inertial>
-  </link> -->
+     <xacro:box_inertia x="1.0" y="1.3" z="2." mass="40"/>
+     </inertial>
+  </link>
+    <!-- Joints of Rockbreaker Arm -->
   <joint name="joint_base_rockbreaker" type="revolute" >
     <axis xyz="0 0 1"/>
-    <limit effort="1000000" lower="-1.57" upper="1.57" velocity="10"/>
+    <limit effort="1000000" lower="-1.57" upper="1.57" velocity="1"/>
     <parent link="rockbreaker_base" />
     <child link="rockbreaker_baserotatoria"  />
@@ -227,5 +138,5 @@
   <joint name="joint_brazoa" type="revolute" >
     <axis xyz="1 0 0"/>
-    <limit effort="1000000" lower="-3.14" upper="3.14" velocity="10"/>
+    <limit effort="1000000" lower="-2.14" upper="2.14" velocity="1"/>
     <parent link="rockbreaker_baserotatoria" />
     <child link="brazo_a" />
@@ -235,5 +146,5 @@
   <joint name="joint_brazob" type="revolute" >
     <axis xyz="1 0 0"/>
-    <limit effort="100000" lower="-3.14" upper="3.14" velocity="10"/>
+    <limit effort="100000" lower="-2.14" upper="2.14" velocity="1"/>
     <parent link="brazo_a" />
     <child link="brazo_b" />
@@ -243,5 +154,5 @@
   <joint name="joint_hammer" type="revolute" >
     <axis xyz="1 0 0"/>
-    <limit effort="100000" lower="-3.14" upper="3.14" velocity="10"/>
+    <limit effort="100000" lower="-2.14" upper="2.14" velocity="1"/>
     <parent link="brazo_b" />
     <child link="h_hammer" />
@@ -249,18 +160,12 @@
     <dynamics damping="${damping_value}" friction="${friction_value}"/>
   </joint>
-  <!-- <joint name="joint_punta" type="revolute" >
-    <axis xyz="0 0 1"/>
-    <limit effort="100000.0" lower="0.0" upper="3.1415" velocity="10000.0"/>
-    <parent link="h_hammer" />
-    <child link="h_punta" />
-    <origin xyz="0.425 -1.65 -1.88" rpy="0 0 0" />
-  </joint> -->
+  <!-- Transmission of Joints -->
   <transmission name="tran1">
     <type>transmission_interface/SimpleTransmission</type>
     <joint name="joint_base_rockbreaker">
-      <hardwareInterface>hardware_interface/EffortJointInterface</hardwareInterface>
+      <hardwareInterface>hardware_interface/PositionJointInterface</hardwareInterface>
     </joint>
     <actuator name="motor1">
-      <hardwareInterface>hardware_interface/EffortJointInterface</hardwareInterface>
+      <hardwareInterface>hardware_interface/PositionJointInterface</hardwareInterface>
       <mechanicalReduction>1</mechanicalReduction>
     </actuator>
@@ -269,8 +174,8 @@
     <type>transmission_interface/SimpleTransmission</type>
     <joint name="joint_brazoa">
-      <hardwareInterface>hardware_interface/EffortJointInterface</hardwareInterface>
+      <hardwareInterface>hardware_interface/PositionJointInterface</hardwareInterface>
     </joint>
     <actuator name="motor2">
-      <hardwareInterface>hardware_interface/EffortJointInterface</hardwareInterface>
+      <hardwareInterface>hardware_interface/PositionJointInterface</hardwareInterface>
       <mechanicalReduction>1</mechanicalReduction>
     </actuator>
@@ -279,8 +184,8 @@
     <type>transmission_interface/SimpleTransmission</type>
     <joint name="joint_brazob">
-      <hardwareInterface>hardware_interface/EffortJointInterface</hardwareInterface>
+      <hardwareInterface>hardware_interface/PositionJointInterface</hardwareInterface>
     </joint>
     <actuator name="motor3">
-      <hardwareInterface>hardware_interface/EffortJointInterface</hardwareInterface>
+      <hardwareInterface>hardware_interface/PositionJointInterfacee</hardwareInterface>
       <mechanicalReduction>1</mechanicalReduction>
     </actuator>
@@ -289,111 +194,15 @@
     <type>transmission_interface/SimpleTransmission</type>
     <joint name="joint_hammer">
-      <hardwareInterface>hardware_interface/EffortJointInterface</hardwareInterface>
+      <hardwareInterface>hardware_interface/PositionJointInterface</hardwareInterface>
     </joint>
     <actuator name="motor4">
-      <hardwareInterface>hardware_interface/EffortJointInterface</hardwareInterface>
-      <mechanicalReduction>1</mechanicalReduction>
-    </actuator>
-  </transmission>
-  <!--
-  <xacro:include filename="$(find velodyne_description)/urdf/VLP-16.urdf.xacro"/>
-  <xacro:VLP-16 parent="excavator_base" name="velodyne" topic="/velodyne_points" organize_cloud="${organize_cloud}" hz="10" samples="440" gpu="${gpu}" >
-    <origin xyz="1 2.7 1.2" rpy="0 0 0" />
-  </xacro:VLP-16>
-  -->
-  <!-- <xacro:include filename=rockbreaker)/urdf/HDL-32E.urdf.xacro"/> -->
-  <!-- <xacro:include filename="$(find lidar_description)/urdf/OS0-64.urdf.xacro"/>
-   <xacro:OS0-64 parent="rockbreaker_base" name="os0_sensor" topic="/os0_cloud_node/points"  hz="10" samples="512" >
-    <origin xyz="3 -13 0" rpy="0 0 1.57" />
-  </xacro:OS0-64> -->
-  <!-- <xacro:include filename=rockbreaker)/urdf/stereo_camera.urdf.xacro"/>
-  <xacro:include filename=rockbreaker)/urdf/VLP-16.urdf.xacro"/>
-  <xacro:stereo_camera_sensor parent="excavator_base" name="camera_front" >
-    <origin xyz="0.8 0 1.5" rpy="0 0 ${-M_PI}" />
-  </xacro:stereo_camera_sensor> -->
-  <!--
-  <xacro:HDL-32E parent="excavator_base" name="velodyne_top" topic="/top/velodyne_points2" organize_cloud="${organize_cloud}" hz="10" samples="220" min_angle="${-M_PI}" max_angle="${M_PI}" gpu="${gpu}" >
-    <origin xyz="0 0 2.8" rpy="0 0 0" />
-  </xacro:HDL-32E>
-  <xacro:camera_sensor parent="excavator_base" name="camera_left_front" >
-    <origin xyz="-0.8 2.7 1.2" rpy="0 0 ${M_PI/2}" />
-  </xacro:camera_sensor>
-  <xacro:camera_sensor parent="excavator_base" name="camera_left_back" >
-    <origin xyz="-0.8 -3 1.2" rpy="0 0 ${-M_PI/2}" />
-  </xacro:camera_sensor>
-  <xacro:camera_sensor parent="excavator_base" name="camera_right_back" >
-    <origin xyz="0.8 -3 1.2" rpy="0 0 ${-M_PI/2}" />
-  </xacro:camera_sensor>
-  -->
-  <!-- <link name="camera_link">
-    <visual>
-      <origin xyz="0 0 0" rpy="0 0 0"/>
-      <geometry>
-        <box size="1 1 1"/>
-      </geometry>
-    </visual>
-    <collision>
-      <origin xyz="0 0 0" rpy="0 0 0"/>
-      <geometry>
-        <box size="1 1 1"/>
-      </geometry>
-    </collision>
-    <inertial>
-      <origin xyz="0 0 0" rpy="0 0 0"/>
-      <mass value="0.035"/>
-      <inertia ixx="0.001"  ixy="0"  ixz="0" iyy="0.001" iyz="0" izz="0.001" />
-    </inertial>
-  </link>
-  <joint name="camera_joint" type="fixed">
-    <parent link="rockbreaker_baserotatoria"/>
-    <child link="camera_link"/>
-    <origin xyz="1 1 1" rpy="0 0 0"/>
-  </joint>
-  <link name="camera_depth_frame"/>
-  <joint name="camera_depth_joint" type="fixed">
-    <origin xyz="0 0 0" rpy="${-pi/2} 0 ${-pi/2}"/>
-    <parent link="camera_link"/>
-    <child link="camera_depth_frame"/>
-  </joint>
-  <gazebo reference="camera_link">
-  <sensor name="depth_camera" type="depth">
-    <update_rate>20</update_rate>
-    <camera>
-      <horizontal_fov>1.047198</horizontal_fov>
-      <image>
-        <width>640</width>
-        <height>480</height>
-        <format>R8G8B8</format>
-      </image>
-      <clip>
-        <near>0.05</near>
-        <far>3</far>
-      </clip>
-    </camera>
-    <plugin name="depth_camera_controller" filename="libgazebo_ros_openni_kinect.so">
-      <baseline>0.2</baseline>
-      <alwaysOn>true</alwaysOn>
-      <updateRate>1.0</updateRate>
-      <cameraName>kine_ir</cameraName>
-      <imageTopicName>/kine/color/image_raw</imageTopicName>
-      <cameraInfoTopicName>/kine/color/camera_info</cameraInfoTopicName>
-      <depthImageTopicName>/kine/depth/image_raw</depthImageTopicName>
-      <depthImageInfoTopicName>/kine/depth/camera_info</depthImageInfoTopicName>
-      <pointCloudTopicName>/kine/depth/points</pointCloudTopicName>
-      <frameName>kine_frame</frameName>
-      <pointCloudCutoff>0.5</pointCloudCutoff>
-      <pointCloudCutoffMax>3.0</pointCloudCutoffMax>
-      <distortionK1>0.00000001</distortionK1>
-      <distortionK2>0.00000001</distortionK2>
-      <distortionK3>0.00000001</distortionK3>
-      <distortionT1>0.00000001</distortionT1>
-      <distortionT2>0.00000001</distortionT2>
-      <CxPrime>0</CxPrime>
-      <Cx>0</Cx>
-      <Cy>0</Cy>
-      <focalLength>0</focalLength>
-      <hackBaseline>0</hackBaseline>
-    </plugin>
-  </sensor>
-</gazebo> -->
+      <hardwareInterface>hardware_interface/PositionJointInterface</hardwareInterface>
+      <mechanicalReduction>1</mechanicalReduction>
+    </actuator>
+  </transmission>
+  <!-- Lidar OS1-64 -->
+  <xacro:include filename="$(find lidar_description)/urdf/OS1-64.urdf.xacro"/>
+  <xacro:OS1-64 parent="rockbreaker_base" name="OS1-64" topic="/os1_cloud_node/points"  samples="256" >
+    <origin xyz="-3.92 -9 1.1" rpy="0 0 2.57" />
+  </xacro:OS1-64>
 </robot>
